File: board/board.kicad_pcb (KiCad board)
At the start: 2 copper layers, 21 x 13 mm, 1 part

Commit message: initial
Parts:
- added C1: 10uF, Capacitor_SMD:C_0402_1005Metric, F.Cu at (147.8, 122.3)
- added C10: 1uF, Capacitor_SMD:C_0402_1005Metric, F.Cu at (153.2, 117.7)
- added C11: 1uF, Capacitor_SMD:C_0402_1005Metric, F.Cu at (152.7, 123.7)
- added C12: 1uF, Capacitor_SMD:C_0402_1005Metric, F.Cu at (147.8, 120.5)
- added C13: 1uF, Capacitor_SMD:C_0402_1005Metric, F.Cu at (147.8, 119.6)
- added C14: 10uF, Capacitor_SMD:C_0402_1005Metric, F.Cu at (148.3, 118.2)
- added C15: 10uF, Capacitor_SMD:C_0402_1005Metric, F.Cu at (150.2, 118.2)
- added C16: 1uF, Capacitor_SMD:C_0402_1005Metric, F.Cu at (147.3, 118.2)
- added C17: 1uF, Capacitor_SMD:C_0402_1005Metric, F.Cu at (149.2, 118.2)
- added C18: 1uF, Capacitor_SMD:C_0402_1005Metric, F.Cu at (153.2, 118.7)
- added C19: 1uF, Capacitor_SMD:C_0402_1005Metric, F.Cu at (153.1, 122.1)
- added C2: 22pF, Capacitor_SMD:C_0402_1005Metric, F.Cu at (145.0, 113.0)
- added C3: 22pF, Capacitor_SMD:C_0402_1005Metric, F.Cu at (149.5, 113.0)
- added C4: 10uF, Capacitor_SMD:C_0402_1005Metric, F.Cu at (146.4, 117.7)
- added C5: 10uF, Capacitor_SMD:C_0402_1005Metric, F.Cu at (151.2, 118.2)
- added C6: 1uF, Capacitor_SMD:C_0402_1005Metric, F.Cu at (150.6, 123.7)
- added C7: 1uF, Capacitor_SMD:C_0402_1005Metric, F.Cu at (148.4, 123.7)
- added C8: 1uF, Capacitor_SMD:C_0402_1005Metric, F.Cu at (153.1, 120.2)
- added C9: 1uF, Capacitor_SMD:C_0402_1005Metric, F.Cu at (153.1, 121.2)
- added FB1: Ferrite_Bead_Small, Inductor_SMD:L_0603_1608Metric, F.Cu at (147.2, 116.0)
- added FB2: Ferrite_Bead_Small, Inductor_SMD:L_0603_1608Metric, F.Cu at (150.2, 116.0)
- added IC1: RTL8305NB-CG, b118:QFN40PEDITED, B.Cu at (150.4, 121.0)
- added J1: 001_I2C, on_edge:on_edge_2x05_device, F.Cu at (140.0, 97.0)
- added J2: 019_100BASE-T_with_CT, on_edge:on_edge_2x05_host, F.Cu at (161.0, 113.0)
- added J3: 019_100BASE-T_with_CT, on_edge:on_edge_2x05_host, F.Cu at (161.0, 129.0)
- added J4: 019_100BASE-T_with_CT, on_edge:on_edge_2x05_host, F.Cu at (161.0, 145.0)
- added J5: 019_100BASE-T_with_CT, on_edge:on_edge_2x05_host, F.Cu at (161.0, 161.0)
- added J6: 019_100BASE-T_with_CT, on_edge:on_edge_2x05_host, F.Cu at (161.0, 97.0)
- added R1: 10k, Resistor_SMD:R_0603_1608Metric, F.Cu at (147.2, 124.3)
- added R10: d.n.p, Resistor_SMD:R_0402_1005Metric, F.Cu at (144.0, 121.8)
- added R11: 1k, Resistor_SMD:R_0603_1608Metric, F.Cu at (141.5, 123.5)
- added R12: d.n.p, Resistor_SMD:R_0402_1005Metric, F.Cu at (144.0, 123.8)
- added R13: 1k, Resistor_SMD:R_0603_1608Metric, F.Cu at (141.5, 125.0)
- added R14: d.n.p, Resistor_SMD:R_0402_1005Metric, F.Cu at (144.0, 124.8)
- added R2: 2.49k, Resistor_SMD:R_0603_1608Metric, F.Cu at (151.5, 114.4)
- added R3: 1k, Resistor_SMD:R_0603_1608Metric, F.Cu at (141.5, 117.5)
- added R4: d.n.p, Resistor_SMD:R_0402_1005Metric, F.Cu at (144.0, 117.8)
- added R5: 1k, Resistor_SMD:R_0603_1608Metric, F.Cu at (141.5, 119.0)
- added R6: d.n.p, Resistor_SMD:R_0402_1005Metric, F.Cu at (144.0, 118.8)
- added R7: 1k, Resistor_SMD:R_0603_1608Metric, F.Cu at (141.5, 120.5)
- added R8: d.n.p, Resistor_SMD:R_0402_1005Metric, F.Cu at (144.0, 120.8)
- added R9: 1k, Resistor_SMD:R_0603_1608Metric, F.Cu at (141.5, 122.0)
- added Y1: 25Mhz, Crystal:Crystal_SMD_2520-4Pin_2.5x2.0mm, F.Cu at (147.3, 113.6)
- moved LOGO1 63.2 mm to (145.6, 162.1)
Routing:
- net +3.3V: track 0.00 -> 146.5 mm, vias 0 -> 13
- net +5V: track 0.00 -> 103.3 mm, vias 0 -> 7
- net GND: track 0.00 -> 79.0 mm, vias 0 -> 64
- net /switch/TXP4: track 0.00 -> 47.0 mm, vias 0 -> 1
- net /switch/TXM4: track 0.00 -> 46.9 mm, vias 0 -> 1
- net /switch/RXM4: track 0.00 -> 41.8 mm, vias 0 -> 1
- net /switch/RXP4: track 0.00 -> 40.8 mm, vias 0 -> 1
- net /switch/1.0V: track 0.00 -> 40.7 mm, vias 0 -> 6
- net /switch/~{RESET}: track 0.00 -> 40.5 mm, vias 0 -> 1
- net /switch/SDA: track 0.00 -> 38.9 mm, vias 0 -> 1
- net /switch/SCL: track 0.00 -> 37.9 mm, vias 0 -> 1
- net /switch/TXP3: track 0.00 -> 29.5 mm, vias 0 -> 1
- net /switch/TXM3: track 0.00 -> 28.9 mm, vias 0 -> 1
- net /switch/RXP0: track 0.00 -> 27.3 mm, vias 0 -> 1
- net /switch/RXM0: track 0.00 -> 26.3 mm, vias 0 -> 1
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- added copper zone on In1.Cu, net +3.3V
- added copper zone on B.Cu, net GND
- added copper zone on F.Cu, net GND
- added copper zone on In2.Cu, net GND
Other:
- board size 21 x 13 mm -> 21 x 78 mm
- copper layers 2 -> 4
- board text added: "osf.001"
- board text added: "osf.019"
- board text added: "osf.b118.v1.0"
